File: sources/PA-circuit.kicad_sch (KiCad schematic)
At the start: 26 parts, among them J2 Conn_01x04_Female, J3 Conn_01x01_Female, U1 MMZ09332BT1, U2 133-3701-311

Commit message: fixing designations
Parts:
- renumbered 1 to J1, U2 to J2, J2 to J3, J3 to J4
Changed lines of the file:
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@@
 		(rev "v0.0")
 		(company "SpaceLab")
-		(comment 1 "Author: Vitória Beatriz Bianchin <vitoriabbianchin@gmail.com>")
+		(comment 1 "Vitória Beatriz Bianchin <vitoriabbianchin@gmail.com>")
 	)
 	(junction
@@
 		(dnp no)
 		(fields_autoplaced yes)
-		(property "Reference" "U2"
+		(property "Reference" "J2"
 			(at 179.07 44.45 0)
 			(effects
@@
 			(project ""
 				(path "/aef50ecb-106b-43ce-b327-8f771253a940"
-					(reference "U2")
+					(reference "J2")
 					(unit 1)
 				)
@@
 		(dnp no)
 		(fields_autoplaced yes)
-		(property "Reference" "J3"
+		(property "Reference" "J4"
 			(at 52.07 110.4899 0)
 			(effects
@@
 			(project ""
 				(path "/aef50ecb-106b-43ce-b327-8f771253a940"
-					(reference "J3")
+					(reference "J4")
 					(unit 1)
 				)
@@
 		(dnp no)
 		(fields_autoplaced yes)
-		(property "Reference" "1"
+		(property "Reference" "J1"
 			(at 38.1 62.23 0)
 			(effects
@@
 			(project ""
 				(path "/aef50ecb-106b-43ce-b327-8f771253a940"
-					(reference "1")
+					(reference "J1")
 					(unit 1)
 				)
@@
 		(dnp no)
 		(fields_autoplaced yes)
-		(property "Reference" "J2"
+		(property "Reference" "J3"
 			(at 57.15 92.7099 0)
 			(effects
@@
 			(project ""
 				(path "/aef50ecb-106b-43ce-b327-8f771253a940"
-					(reference "J2")
+					(reference "J3")
 					(unit 1)
 				)

Commit message: updating rf connector and lib
Parts:
- J1, J2: footprint 133-3701-311:133-3701-311 -> 2016504-1:2016504-1
Changed lines of the file:
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@@
 			)
 		)
-		(property "Footprint" "133-3701-311:133-3701-311"
+		(property "Footprint" "2016504-1:2016504-1"
 			(at 168.91 57.15 0)
 			(effects
@@
 			)
 		)
-		(property "Footprint" "133-3701-311:133-3701-311"
+		(property "Footprint" "2016504-1:2016504-1"
 			(at 48.26 80.01 0)
 			(effects

Commit message: finishing layout
Parts:
- J3: value Conn_01x04_Female -> Conn_01x05; footprint Connector_PinHeader_2.54mm:PinHeader_1x04_P2.54mm_Vertical -> Connector_PinHeader_2.54mm:PinHeader_1x05_P2.54mm_Vertical
- renumbered C3 to C1, C2 to C10, C6 to C2, C7 to C3, C5 to C4, C8 to C5, C4 to C6, C1 to C7, C9 to C8, C10 to C9, H4 to H1, H1 to H3, H3 to H4, J4 to J2, J2 to J4
